File: hardware/sd-net.kicad_sch (KiCad schematic)
At the start: 11 parts, among them U1 GL823K-HCY04

Commit message: emit KiCad 10 schematic format and stop designator text colliding
Two fixes from opening the schematic in the GUI for the first time.

KiCad 10 writes .kicad_sch version 20260306; the generator was emitting the 9.0
format 20250114, which loaded but triggered an "older version of KiCad"
conversion banner. Discovered the number by running kicad-cli sch upgrade, and
the generator now emits it directly -- ERC and the netlist check still pass.

Reference and value text was placed at a fixed offset tuned for the tall custom
symbols, which threw R1's and LED1's designators 22.86 mm up into the capacitor
row. Text placement is now per-symbol: above the big parts, to the right for the
two-pin Device symbols whose pins already carry net labels above and below.
Changed lines of the file:
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@@
 (kicad_sch
-	(version 20250114)
+	(version 20260306)
 	(generator "sd-net gen_schematic.py")
 	(generator_version "10.0")
@@
 		(fields_autoplaced yes)
 		(property "Reference" "U1"
-			(at 146.05 77.47 0)
+			(at 146.05 80.00999999999999 0)
 			(effects (font (size 1.27 1.27)))
 		)
 		(property "Value" "GL823K-HCY04"
-			(at 146.05 80.00999999999999 0)
+			(at 146.05 82.55 0)
 			(effects (font (size 1.27 1.27)))
 		)
@@
 		(instances
 			(project "sd-net"
-				(path "/6cf8bc62-746e-415c-82ae-79da5e44ee34"
+				(path "/9081c948-1d60-4f6f-8cc7-11daea454aad"
 					(reference "U1") (unit 1)
 				)
@@
 		(fields_autoplaced yes)
 		(property "Reference" "CARD1"
-			(at 215.9 77.47 0)
+			(at 215.9 78.74 0)
 			(effects (font (size 1.27 1.27)))
 		)
 		(property "Value" "SD-006M"
-			(at 215.9 80.00999999999999 0)
+			(at 215.9 81.28 0)
 			(effects (font (size 1.27 1.27)))
 		)
@@
 		(instances
 			(project "sd-net"
-				(path "/6cf8bc62-746e-415c-82ae-79da5e44ee34"
+				(path "/9081c948-1d60-4f6f-8cc7-11daea454aad"
 					(reference "CARD1") (unit 1)
 				)
@@
 		(fields_autoplaced yes)
 		(property "Reference" "USB1"
-			(at 68.58 77.47 0)
+			(at 68.58 87.63 0)
 			(effects (font (size 1.27 1.27)))
 		)
 		(property "Value" "AM90"
-			(at 68.58 80.00999999999999 0)
+			(at 68.58 90.17 0)
 			(effects (font (size 1.27 1.27)))
 		)
@@
 		(instances
 			(project "sd-net"
-				(path "/6cf8bc62-746e-415c-82ae-79da5e44ee34"
+				(path "/9081c948-1d60-4f6f-8cc7-11daea454aad"
 					(reference "USB1") (unit 1)
 				)
@@
 		(fields_autoplaced yes)
 		(property "Reference" "C1"
-			(at 68.58 125.73 0)
-			(effects (font (size 1.27 1.27)))
+			(at 72.39 147.32 0)
+			(effects (font (size 1.27 1.27)) (justify left))
 		)
 		(property "Value" "10uF"
-			(at 68.58 128.27 0)
-			(effects (font (size 1.27 1.27)))
+			(at 72.39 149.85999999999999 0)
+			(effects (font (size 1.27 1.27)) (justify left))
 		)
 		(property "Footprint" "Capacitor_SMD:C_0805_2012Metric"
@@
 		(instances
 			(project "sd-net"
-				(path "/6cf8bc62-746e-415c-82ae-79da5e44ee34"
+				(path "/9081c948-1d60-4f6f-8cc7-11daea454aad"
 					(reference "C1") (unit 1)
 				)
@@
 		(fields_autoplaced yes)
 		(property "Reference" "C4"
-			(at 88.9 125.73 0)
-			(effects (font (size 1.27 1.27)))
+			(at 92.71000000000001 147.32 0)
+			(effects (font (size 1.27 1.27)) (justify left))
 		)
 		(property "Value" "100nF"
-			(at 88.9 128.27 0)
-			(effects (font (size 1.27 1.27)))
+			(at 92.71000000000001 149.85999999999999 0)
+			(effects (font (size 1.27 1.27)) (justify left))
 		)
 		(property "Footprint" "Capacitor_SMD:C_0603_1608Metric"
@@
 		(instances
 			(project "sd-net"
-				(path "/6cf8bc62-746e-415c-82ae-79da5e44ee34"
+				(path "/9081c948-1d60-4f6f-8cc7-11daea454aad"
 					(reference "C4") (unit 1)
 				)
@@
 		(fields_autoplaced yes)
 		(property "Reference" "C2"
-			(at 109.22 125.73 0)
-			(effects (font (size 1.27 1.27)))
+			(at 113.03 147.32 0)
+			(effects (font (size 1.27 1.27)) (justify left))
 		)
 		(property "Value" "10uF"
-			(at 109.22 128.27 0)
-			(effects (font (size 1.27 1.27)))
+			(at 113.03 149.85999999999999 0)
+			(effects (font (size 1.27 1.27)) (justify left))
 		)
 		(property "Footprint" "Capacitor_SMD:C_0805_2012Metric"
@@
 		(instances
 			(project "sd-net"
-				(path "/6cf8bc62-746e-415c-82ae-79da5e44ee34"
+				(path "/9081c948-1d60-4f6f-8cc7-11daea454aad"
 					(reference "C2") (unit 1)
 				)
@@
 		(fields_autoplaced yes)
 		(property "Reference" "C5"
-			(at 129.54 125.73 0)
-			(effects (font (size 1.27 1.27)))
+			(at 133.35 147.32 0)
+			(effects (font (size 1.27 1.27)) (justify left))
 		)
 		(property "Value" "100nF"
-			(at 129.54 128.27 0)
-			(effects (font (size 1.27 1.27)))
+			(at 133.35 149.85999999999999 0)
+			(effects (font (size 1.27 1.27)) (justify left))
 		)
 		(property "Footprint" "Capacitor_SMD:C_0603_1608Metric"
@@
 		(instances
 			(project "sd-net"
-				(path "/6cf8bc62-746e-415c-82ae-79da5e44ee34"
+				(path "/9081c948-1d60-4f6f-8cc7-11daea454aad"
 					(reference "C5") (unit 1)
 				)
@@
 		(fields_autoplaced yes)
 		(property "Reference" "C6"
-			(at 149.86 125.73 0)
-			(effects (font (size 1.27 1.27)))
+			(at 153.67000000000002 147.32 0)
+			(effects (font (size 1.27 1.27)) (justify left))
 		)
 		(property "Value" "100nF"
-			(at 149.86 128.27 0)
-			(effects (font (size 1.27 1.27)))
+			(at 153.67000000000002 149.85999999999999 0)
+			(effects (font (size 1.27 1.27)) (justify left))
 		)
 		(property "Footprint" "Capacitor_SMD:C_0603_1608Metric"
@@
 		(instances
 			(project "sd-net"
-				(path "/6cf8bc62-746e-415c-82ae-79da5e44ee34"
+				(path "/9081c948-1d60-4f6f-8cc7-11daea454aad"
 					(reference "C6") (unit 1)
 				)
@@
 		(fields_autoplaced yes)
 		(property "Reference" "C3"
-			(at 170.18 125.73 0)
-			(effects (font (size 1.27 1.27)))
+			(at 173.99 147.32 0)
+			(effects (font (size 1.27 1.27)) (justify left))
 		)
 		(property "Value" "10uF"
-			(at 170.18 128.27 0)
-			(effects (font (size 1.27 1.27)))
+			(at 173.99 149.85999999999999 0)
+			(effects (font (size 1.27 1.27)) (justify left))
 		)
 		(property "Footprint" "Capacitor_SMD:C_0805_2012Metric"
@@
 		(instances
 			(project "sd-net"
-				(path "/6cf8bc62-746e-415c-82ae-79da5e44ee34"
+				(path "/9081c948-1d60-4f6f-8cc7-11daea454aad"
 					(reference "C3") (unit 1)
 				)
@@
 		(fields_autoplaced yes)
 		(property "Reference" "R1"
-			(at 68.58 151.13 0)
-			(effects (font (size 1.27 1.27)))
+			(at 72.39 172.72 0)
+			(effects (font (size 1.27 1.27)) (justify left))
 		)
 		(property "Value" "220"
-			(at 68.58 153.67000000000002 0)
-			(effects (font (size 1.27 1.27)))
+			(at 72.39 175.26 0)
+			(effects (font (size 1.27 1.27)) (justify left))
 		)
 		(property "Footprint" "Resistor_SMD:R_0603_1608Metric"
@@
 		(instances
 			(project "sd-net"
-				(path "/6cf8bc62-746e-415c-82ae-79da5e44ee34"
+				(path "/9081c948-1d60-4f6f-8cc7-11daea454aad"
 					(reference "R1") (unit 1)
 				)
@@
 		(fields_autoplaced yes)
 		(property "Reference" "LED1"
-			(at 96.52 151.13 0)
-			(effects (font (size 1.27 1.27)))
+			(at 100.33 172.72 0)
+			(effects (font (size 1.27 1.27)) (justify left))
 		)
 		(property "Value" "12-215SYGC"
-			(at 96.52 153.67000000000002 0)
-			(effects (font (size 1.27 1.27)))
+			(at 100.33 175.26 0)
+			(effects (font (size 1.27 1.27)) (justify left))
 		)
 		(property "Footprint" "LED_SMD:LED_0603_1608Metric"
@@
 		(instances
 			(project "sd-net"
-				(path "/6cf8bc62-746e-415c-82ae-79da5e44ee34"
+				(path "/9081c948-1d60-4f6f-8cc7-11daea454aad"
 					(reference "LED1") (unit 1)
 				)
@@
 		(fields_autoplaced yes)
 		(property "Reference" "#FLG01"
-			(at 60.96 167.64 0)
-			(effects (font (size 1.27 1.27)))
+			(at 64.77 189.23 0)
+			(effects (font (size 1.27 1.27)) (justify left))
 		)
 		(property "Value" "PWR_FLAG"
-			(at 60.96 170.18 0)
-			(effects (font (size 1.27 1.27)))
+			(at 64.77 191.76999999999998 0)
+			(effects (font (size 1.27 1.27)) (justify left))
 		)
 		(property "Footprint" ""
@@
 		(instances
 			(project "sd-net"
-				(path "/6cf8bc62-746e-415c-82ae-79da5e44ee34"
+				(path "/9081c948-1d60-4f6f-8cc7-11daea454aad"
 					(reference "#FLG01") (unit 1)
 				)

Commit message: fix pin-side mapping for horizontal symbols
A pin's angle gives the direction from its connection point toward the symbol
body, so the connection sits on the opposite side. The stock-symbol path only
distinguished 270 from everything else, which is right for the vertical
Device:C and Device:R but wrong for Device:LED, whose pins are horizontal
(0/180). LED1 ended up with both net labels rotated vertically and its
designator text overlapping LED_A.

Now maps all four angles, and LED1's text sits above the part rather than to
the right where its own pin label lives. ERC and the netlist check still pass.
Changed lines of the file:
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@@
 		(instances
 			(project "sd-net"
-				(path "/9081c948-1d60-4f6f-8cc7-11daea454aad"
+				(path "/454a1c01-2ff6-4d72-bb44-9726975a5cb6"
 					(reference "U1") (unit 1)
 				)
@@
 		(instances
 			(project "sd-net"
-				(path "/9081c948-1d60-4f6f-8cc7-11daea454aad"
+				(path "/454a1c01-2ff6-4d72-bb44-9726975a5cb6"
 					(reference "CARD1") (unit 1)
 				)
@@
 		(instances
 			(project "sd-net"
-				(path "/9081c948-1d60-4f6f-8cc7-11daea454aad"
+				(path "/454a1c01-2ff6-4d72-bb44-9726975a5cb6"
 					(reference "USB1") (unit 1)
 				)
@@
 		(instances
 			(project "sd-net"
-				(path "/9081c948-1d60-4f6f-8cc7-11daea454aad"
+				(path "/454a1c01-2ff6-4d72-bb44-9726975a5cb6"
 					(reference "C1") (unit 1)
 				)
@@
 		(instances
 			(project "sd-net"
-				(path "/9081c948-1d60-4f6f-8cc7-11daea454aad"
+				(path "/454a1c01-2ff6-4d72-bb44-9726975a5cb6"
 					(reference "C4") (unit 1)
 				)
@@
 		(instances
 			(project "sd-net"
-				(path "/9081c948-1d60-4f6f-8cc7-11daea454aad"
+				(path "/454a1c01-2ff6-4d72-bb44-9726975a5cb6"
 					(reference "C2") (unit 1)
 				)
@@
 		(instances
 			(project "sd-net"
-				(path "/9081c948-1d60-4f6f-8cc7-11daea454aad"
+				(path "/454a1c01-2ff6-4d72-bb44-9726975a5cb6"
 					(reference "C5") (unit 1)
 				)
@@
 		(instances
 			(project "sd-net"
-				(path "/9081c948-1d60-4f6f-8cc7-11daea454aad"
+				(path "/454a1c01-2ff6-4d72-bb44-9726975a5cb6"
 					(reference "C6") (unit 1)
 				)
@@
 		(instances
 			(project "sd-net"
-				(path "/9081c948-1d60-4f6f-8cc7-11daea454aad"
+				(path "/454a1c01-2ff6-4d72-bb44-9726975a5cb6"
 					(reference "C3") (unit 1)
 				)
@@
 		(instances
 			(project "sd-net"
-				(path "/9081c948-1d60-4f6f-8cc7-11daea454aad"
+				(path "/454a1c01-2ff6-4d72-bb44-9726975a5cb6"
 					(reference "R1") (unit 1)
 				)
@@
 		(fields_autoplaced yes)
 		(property "Reference" "LED1"
-			(at 100.33 172.72 0)
-			(effects (font (size 1.27 1.27)) (justify left))
+			(at 96.52 168.91 0)
+			(effects (font (size 1.27 1.27)))
 		)
 		(property "Value" "12-215SYGC"
-			(at 100.33 175.26 0)
-			(effects (font (size 1.27 1.27)) (justify left))
+			(at 96.52 171.45 0)
+			(effects (font (size 1.27 1.27)))
 		)
 		(property "Footprint" "LED_SMD:LED_0603_1608Metric"
@@
 		(instances
 			(project "sd-net"
-				(path "/9081c948-1d60-4f6f-8cc7-11daea454aad"
+				(path "/454a1c01-2ff6-4d72-bb44-9726975a5cb6"
 					(reference "LED1") (unit 1)
 				)
@@
 		(instances
 			(project "sd-net"
-				(path "/9081c948-1d60-4f6f-8cc7-11daea454aad"
+				(path "/454a1c01-2ff6-4d72-bb44-9726975a5cb6"
 					(reference "#FLG01") (unit 1)
 				)
@@
 	)
 	(wire
-		(pts (xy 100.33 173.99) (xy 100.33 177.8))
+		(pts (xy 100.33 173.99) (xy 104.14 173.99))
 		(stroke (width 0) (type default))
 	)
 	(global_label "LED_A"
 		(shape bidirectional)
-		(at 100.33 177.8 270)
-		(fields_autoplaced yes)
-		(effects (font (size 1.27 1.27)) (justify left))
-	)
-	(wire
-		(pts (xy 92.71 173.99) (xy 92.71 177.8))
+		(at 104.14 173.99 0)
+		(fields_autoplaced yes)
+		(effects (font (size 1.27 1.27)) (justify left))
+	)
+	(wire
+		(pts (xy 92.71 173.99) (xy 88.89999999999999 173.99))
 		(stroke (width 0) (type default))
 	)
 	(global_label "LED_K"
 		(shape bidirectional)
-		(at 92.71 177.8 270)
-		(fields_autoplaced yes)
-		(effects (font (size 1.27 1.27)) (justify left))
-	)
-	(wire
+		(at 88.89999999999999 173.99 180)
+		(fields_autoplaced yes)
+		(effects (font (size 1.27 1.27)) (justify right))
+	)
+	(wire

Commit message: add C7 and C8 so all four power rails get proper decoupling
Rev 1.5's six capacitors stretch to three rails, not the four the fixed
topology needs: VCARD had bulk but no high-frequency cap, and VDDA had a single
100 nF and no bulk. C7 (VCARD) and C8 (VDDA) are the same 100 nF 0603 as
C4/C5/C6, LCSC C14663, so no new line item -- 11 placements becomes 13.

The capacitor row in the schematic is regrouped by rail. tools/verify_netlist.py
now separates pads that were floating in rev 1.5 from parts that did not exist
in it, so the two show up honestly in the diff rather than both reading as
'newly connected'. ERC clean, netlist verified.
Parts:
- added C7, C8: 100nF, Capacitor_SMD:C_0603_1608Metric, symbol Device:C
Connections:
- net GND: now also C7.2, C8.2
- net VCARD: now also C7.1
- net VDDA: now also C8.1
Changed lines of the file:
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@@
 		(instances
 			(project "sd-net"
-				(path "/454a1c01-2ff6-4d72-bb44-9726975a5cb6"
+				(path "/1ebe58e1-8cab-4a64-8f47-26625183a810"
 					(reference "U1") (unit 1)
 				)
@@
 		(instances
 			(project "sd-net"
-				(path "/454a1c01-2ff6-4d72-bb44-9726975a5cb6"
+				(path "/1ebe58e1-8cab-4a64-8f47-26625183a810"
 					(reference "CARD1") (unit 1)
 				)
@@
 		(instances
 			(project "sd-net"
-				(path "/454a1c01-2ff6-4d72-bb44-9726975a5cb6"
+				(path "/1ebe58e1-8cab-4a64-8f47-26625183a810"
 					(reference "USB1") (unit 1)
 				)
@@
 		(instances
 			(project "sd-net"
-				(path "/454a1c01-2ff6-4d72-bb44-9726975a5cb6"
+				(path "/1ebe58e1-8cab-4a64-8f47-26625183a810"
 					(reference "C1") (unit 1)
 				)
@@
 		(instances
 			(project "sd-net"
-				(path "/454a1c01-2ff6-4d72-bb44-9726975a5cb6"
+				(path "/1ebe58e1-8cab-4a64-8f47-26625183a810"
 					(reference "C4") (unit 1)
 				)
@@
 		(instances
 			(project "sd-net"
-				(path "/454a1c01-2ff6-4d72-bb44-9726975a5cb6"
+				(path "/1ebe58e1-8cab-4a64-8f47-26625183a810"
 					(reference "C2") (unit 1)
 				)
@@
 		(instances
 			(project "sd-net"
-				(path "/454a1c01-2ff6-4d72-bb44-9726975a5cb6"
+				(path "/1ebe58e1-8cab-4a64-8f47-26625183a810"
 					(reference "C5") (unit 1)
 				)
@@
 		(instances
 			(project "sd-net"
-				(path "/454a1c01-2ff6-4d72-bb44-9726975a5cb6"
+				(path "/1ebe58e1-8cab-4a64-8f47-26625183a810"
 					(reference "C6") (unit 1)
 				)
@@
 		(dnp no)
 		(fields_autoplaced yes)
+		(property "Reference" "C8"
+			(at 173.99 147.32 0)
+			(effects (font (size 1.27 1.27)) (justify left))
+		)
+		(property "Value" "100nF"
+			(at 173.99 149.85999999999999 0)
+			(effects (font (size 1.27 1.27)) (justify left))
+		)
+		(property "Footprint" "Capacitor_SMD:C_0603_1608Metric"
+			(at 170.18 148.59 0)
+			(effects (font (size 1.27 1.27)) (hide yes))
+		)
+		(property "LCSC" "C14663"
+			(at 170.18 148.59 0)
+			(effects (font (size 1.27 1.27)) (hide yes))
+		)
+		(instances
+			(project "sd-net"
+				(path "/1ebe58e1-8cab-4a64-8f47-26625183a810"
+					(reference "C8") (unit 1)
+				)
+			)
+		)
+	)
+	(symbol
+		(lib_id "Device:C")
+		(at 190.5 148.59 0)
+		(unit 1)
+		(exclude_from_sim no)
+		(in_bom yes)
+		(on_board yes)
+		(dnp no)
+		(fields_autoplaced yes)
 		(property "Reference" "C3"
-			(at 173.99 147.32 0)
+			(at 194.31 147.32 0)
 			(effects (font (size 1.27 1.27)) (justify left))
 		)
 		(property "Value" "10uF"
-			(at 173.99 149.85999999999999 0)
+			(at 194.31 149.85999999999999 0)
 			(effects (font (size 1.27 1.27)) (justify left))
 		)
 		(property "Footprint" "Capacitor_SMD:C_0805_2012Metric"
-			(at 170.18 148.59 0)
+			(at 190.5 148.59 0)
 			(effects (font (size 1.27 1.27)) (hide yes))
 		)
 		(property "LCSC" "C15850"
-			(at 170.18 148.59 0)
-			(effects (font (size 1.27 1.27)) (hide yes))
-		)
-		(instances
-			(project "sd-net"
-				(path "/454a1c01-2ff6-4d72-bb44-9726975a5cb6"
+			(at 190.5 148.59 0)
+			(effects (font (size 1.27 1.27)) (hide yes))
+		)
+		(instances
+			(project "sd-net"
+				(path "/1ebe58e1-8cab-4a64-8f47-26625183a810"
 					(reference "C3") (unit 1)
+				)
+			)
+		)
+	)
+	(symbol
+		(lib_id "Device:C")
+		(at 210.82 148.59 0)
+		(unit 1)
+		(exclude_from_sim no)
+		(in_bom yes)
+		(on_board yes)
+		(dnp no)
+		(fields_autoplaced yes)
+		(property "Reference" "C7"
+			(at 214.63 147.32 0)
+			(effects (font (size 1.27 1.27)) (justify left))
+		)
+		(property "Value" "100nF"
+			(at 214.63 149.85999999999999 0)
+			(effects (font (size 1.27 1.27)) (justify left))
+		)
+		(property "Footprint" "Capacitor_SMD:C_0603_1608Metric"
+			(at 210.82 148.59 0)
+			(effects (font (size 1.27 1.27)) (hide yes))
+		)
+		(property "LCSC" "C14663"
+			(at 210.82 148.59 0)
+			(effects (font (size 1.27 1.27)) (hide yes))
+		)
+		(instances
+			(project "sd-net"
+				(path "/1ebe58e1-8cab-4a64-8f47-26625183a810"
+					(reference "C7") (unit 1)
 				)
 			)
@@
 		(instances
 			(project "sd-net"
-				(path "/454a1c01-2ff6-4d72-bb44-9726975a5cb6"
+				(path "/1ebe58e1-8cab-4a64-8f47-26625183a810"
 					(reference "R1") (unit 1)
 				)
@@
 		(instances
 			(project "sd-net"
-				(path "/454a1c01-2ff6-4d72-bb44-9726975a5cb6"
+				(path "/1ebe58e1-8cab-4a64-8f47-26625183a810"
 					(reference "LED1") (unit 1)
 				)
@@
 		(instances
 			(project "sd-net"
-				(path "/454a1c01-2ff6-4d72-bb44-9726975a5cb6"
+				(path "/1ebe58e1-8cab-4a64-8f47-26625183a810"
 					(reference "#FLG01") (unit 1)
 				)
@@
 	)
 	(wire
+		(pts (xy 170.18 144.78) (xy 170.18 140.97))
+		(stroke (width 0) (type default))
+	)
+	(global_label "VDDA"
+		(shape bidirectional)
+		(at 170.18 140.97 90)
+		(fields_autoplaced yes)
+		(effects (font (size 1.27 1.27)) (justify left))
+	)
+	(wire
 		(pts (xy 128.27 95.25) (xy 124.46000000000001 95.25))
 		(stroke (width 0) (type default))
@@
 	)
 	(wire
-		(pts (xy 170.18 144.78) (xy 170.18 140.97))
+		(pts (xy 190.5 144.78) (xy 190.5 140.97))
 		(stroke (width 0) (type default))
 	)
 	(global_label "VCARD"
 		(shape bidirectional)
-		(at 170.18 140.97 90)
+		(at 190.5 140.97 90)
+		(fields_autoplaced yes)
+		(effects (font (size 1.27 1.27)) (justify left))
+	)
+	(wire
+		(pts (xy 210.82 144.78) (xy 210.82 140.97))
+		(stroke (width 0) (type default))
+	)
+	(global_label "VCARD"
+		(shape bidirectional)
+		(at 210.82 140.97 90)
 		(fields_autoplaced yes)
 		(effects (font (size 1.27 1.27)) (justify left))
@@
 	)
 	(wire
+		(pts (xy 190.5 152.4) (xy 190.5 156.21))
+		(stroke (width 0) (type default))
+	)
+	(global_label "GND"
+		(shape bidirectional)
+		(at 190.5 156.21 270)
+		(fields_autoplaced yes)
+		(effects (font (size 1.27 1.27)) (justify left))
+	)
+	(wire
+		(pts (xy 88.9 152.4) (xy 88.9 156.21))
+		(stroke (width 0) (type default))
+	)
+	(global_label "GND"
+		(shape bidirectional)
+		(at 88.9 156.21 270)
+		(fields_autoplaced yes)
+		(effects (font (size 1.27 1.27)) (justify left))
+	)
+	(wire
+		(pts (xy 129.54 152.4) (xy 129.54 156.21))
+		(stroke (width 0) (type default))
+	)
+	(global_label "GND"
+		(shape bidirectional)
+		(at 129.54 156.21 270)
+		(fields_autoplaced yes)
+		(effects (font (size 1.27 1.27)) (justify left))
+	)
+	(wire
+		(pts (xy 149.86 152.4) (xy 149.86 156.21))
+		(stroke (width 0) (type default))
+	)
+	(global_label "GND"
+		(shape bidirectional)
+		(at 149.86 156.21 270)
+		(fields_autoplaced yes)
+		(effects (font (size 1.27 1.27)) (justify left))
+	)
+	(wire
+		(pts (xy 210.82 152.4) (xy 210.82 156.21))
+		(stroke (width 0) (type default))
+	)
+	(global_label "GND"
+		(shape bidirectional)
+		(at 210.82 156.21 270)
+		(fields_autoplaced yes)
+		(effects (font (size 1.27 1.27)) (justify left))
+	)
+	(wire
 		(pts (xy 170.18 152.4) (xy 170.18 156.21))
 		(stroke (width 0) (type default))
@@
 		(fields_autoplaced yes)
 		(effects (font (size 1.27 1.27)) (justify left))
-	)
-	(wire
-		(pts (xy 88.9 152.4) (xy 88.9 156.21))
-		(stroke (width 0) (type default))
-	)
-	(global_label "GND"
-		(shape bidirectional)
-		(at 88.9 156.21 270)
-		(fields_autoplaced yes)
-		(effects (font (size 1.27 1.27)) (justify left))
-	)
-	(wire
-		(pts (xy 129.54 152.4) (xy 129.54 156.21))
-		(stroke (width 0) (type default))
-	)
-	(global_label "GND"
-		(shape bidirectional)
-		(at 129.54 156.21 270)
-		(fields_autoplaced yes)
-		(effects (font (size 1.27 1.27)) (justify left))
-	)
-	(wire
-		(pts (xy 149.86 152.4) (xy 149.86 156.21))
-		(stroke (width 0) (type default))
-	)
-	(global_label "GND"
-		(shape bidirectional)
-		(at 149.86 156.21 270)
-		(fields_autoplaced yes)
-		(effects (font (size 1.27 1.27)) (justify left))
